File: PCB/submodule/protecciones.kicad_sch (KiCad schematic)
At the start: 35 parts, among them J10 Conn_Coaxial, J11 Conn_Coaxial, J12 Conn_Coaxial, J13 Conn_Coaxial, J14 Conn_Coaxial, J15 Conn_Coaxial, J16 Conn_Coaxial, J17 Conn_Coaxial, J6 ELECT_AUX, J7 Conn_Coaxial, J9 Conn_Coaxial, U3 TPD4E001, U4 TPD4E001, U5 TPD2E001

Commit message: Power supply & TPDs
Parts:
- removed C13, C15: 1nF, symbol Device:C
- removed J10, J11, J12, J13, J14, J15, J16, J17, J7, J9: Conn_Coaxial, Connector_Coaxial:U.FL_Molex_MCRF_73412-0110_Vertical, symbol Connector:Conn_Coaxial
- removed J6: ELECT_AUX, symbol Connector_Generic:Conn_01x12
- removed R12: 39k, symbol Device:R
- removed R13, R15: 2k2, symbol Device:R
- removed U5: TPD2E001, DRL5, symbol TPD2:TPD2E001DRLR
- added C1, C34: 1nF, symbol Device:C
- added R18: 39k, symbol Device:R
- added R19, R21: 2k2, symbol Device:R
- added U8: TPD4E001, DPK6, symbol TPD4:TPD4E001DPKT
Connections:
- net AGND: now also C1.2, C34.2; no longer U3.3 (GND), U4.3 (GND)
- net BIAS_DRV: now also R18.2
- net BIAS_ELEC: now also C1.1, R19.1
- net IN_ELEC: now also R21.2, U8.1 (IO1)
- net IN_REF: now also C34.1, R21.1
- net +5V renamed AVDD
- net AVDD: now also U8.6 (VCC)
- net CH1_IN renamed CH_IN1
- net CH2_IN renamed CH_IN2
- net CH3_IN renamed CH_IN3
- net CH5_IN renamed CH_IN5
- net CH6_IN renamed CH_IN6
- net CH7_IN renamed CH_IN7
- new net: R18.1, R19.2, U8.2 (IO2)
- new net AVSS: U3.3 (GND), U4.3 (GND), U8.3 (GND)
- no-connect marks 1 -> 2
Other:
- note removed: "Mejor lo unificamos a uno de 4 canales, no?"
- note removed: "OJO! Esta debería ser la tensión de alimentación del ADS"

Commit message: draft initial wiring for submodule (pending pin check)
Changed lines of the file:
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@@
 	(wire
 		(pts
-			(xy 25.4 71.12) (xy 29.21 71.12)
+			(xy 29.21 29.21) (xy 33.02 29.21)
 		)
 		(stroke
@@
 	(wire
 		(pts
-			(xy 25.4 74.93) (xy 29.21 74.93)
+			(xy 29.21 33.02) (xy 33.02 33.02)
 		)
 		(stroke
@@
 	)
 	(label "BIAS_ELEC"
-		(at 25.4 71.12 180)
+		(at 29.21 29.21 180)
 		(effects
 			(font
@@
 	)
 	(label "IN_ELEC"
-		(at 25.4 74.93 180)
+		(at 29.21 33.02 180)
 		(effects
 			(font
@@
 	(hierarchical_label "IN_ELEC"
 		(shape input)
-		(at 29.21 74.93 0)
+		(at 33.02 33.02 0)
 		(effects
 			(font
@@
 	(hierarchical_label "BIAS_ELEC"
 		(shape input)
-		(at 29.21 71.12 0)
-		(effects
-			(font
+		(at 33.02 29.21 0)
+		(effects
+			(font

Commit message: fix GPIOs
Other:
- moved on the sheet: C1, C10, C11, C12, C34, C5, C6, C7, C8, C9, R10, R11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

Commit message: fix BIAS (pending ERC & footprints)
Connections:
- net BIAS_DRV: now also C1.1, R19.1; no longer R18.2
- net BIAS_ELEC: now also R18.2; no longer C1.1, R19.1
Changed lines of the file:
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@@
-		)
-	)
-	(label "BIAS_DRV"
-		(at 173.99 77.47 0)
-		(effects
-			(font
-				(size 1.27 1.27)
-			)
-			(justify left bottom)
 		)
 	)
@@
 			)
 			(justify right bottom)
-		)
-	)
-	(label "BIAS_ELEC"
-		(at 242.57 77.47 0)
-		(effects
-			(font
-				(size 1.27 1.27)
-			)
-			(justify left bottom)
 		)
 	)
@@
 		)
 	)
+	(label "BIAS_DRV"
+		(at 242.57 77.47 0)
+		(effects
+			(font
+				(size 1.27 1.27)
+			)
+			(justify left bottom)
+		)
+	)
 	(label "IN1+"
 		(at 139.7 39.37 0)
@@
 		(effects
 			(font
+				(size 1.27 1.27)
+			)
+			(justify left bottom)
+		)
+	)
+	(label "BIAS_ELEC"
+		(at 173.99 77.47 0)
+		(effects
+			(font
