File: PCB/submodule/protecciones.kicad_sch (KiCad schematic)
At the start: 24 parts, among them U3 TPD4E001, U4 TPD4E001, U8 TPD4E001

Commit message: ECR ok
Connections:
- net CH_IN3: no longer R7.2, U3.5 (IO4)
- net CH_IN7: no longer R10.2, U4.5 (IO4)
- new net CH_IN4: R7.2, U3.5 (IO4)
- new net CH_IN8: R10.2, U4.5 (IO4)
Changed lines of the file:
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@@
 	)
 	(junction
-		(at 102.87 78.74)
-		(diameter 0)
-		(color 0 0 0 0)
-	)
-	(junction
 		(at 100.33 78.74)
 		(diameter 0)
@@
 		(color 0 0 0 0)
 	)
-	(junction
-		(at 102.87 139.7)
-		(diameter 0)
-		(color 0 0 0 0)
-	)
 	(no_connect
 		(at 203.2 107.95)
@@
 	(wire
 		(pts
-			(xy 102.87 78.74) (xy 102.87 82.55)
+			(xy 102.87 73.66) (xy 102.87 82.55)
 		)
 		(stroke
@@
 	(wire
 		(pts
-			(xy 31.75 88.9) (xy 41.91 88.9)
-		)
-		(stroke
-			(width 0)
-			(type default)
-		)
-	)
-	(wire
-		(pts
 			(xy 105.41 135.89) (xy 85.09 135.89)
 		)
@@
 	(wire
 		(pts
-			(xy 102.87 73.66) (xy 102.87 78.74)
-		)
-		(stroke
-			(width 0)
-			(type default)
-		)
-	)
-	(wire
-		(pts
 			(xy 208.28 73.66) (xy 208.28 81.28)
 		)
@@
 	(wire
 		(pts
-			(xy 102.87 139.7) (xy 102.87 143.51)
+			(xy 102.87 134.62) (xy 102.87 143.51)
 		)
 		(stroke
@@
 	(wire
 		(pts
-			(xy 102.87 78.74) (xy 107.95 78.74)
+			(xy 100.33 78.74) (xy 107.95 78.74)
 		)
 		(stroke
@@
 	(wire
 		(pts
-			(xy 100.33 78.74) (xy 102.87 78.74)
-		)
-		(stroke
-			(width 0)
-			(type default)
-		)
-	)
-	(wire
-		(pts
 			(xy 132.08 73.66) (xy 132.08 82.55)
 		)
@@
 	(wire
 		(pts
-			(xy 100.33 139.7) (xy 102.87 139.7)
+			(xy 100.33 139.7) (xy 107.95 139.7)
 		)
 		(stroke
@@
 	(wire
 		(pts
-			(xy 102.87 139.7) (xy 107.95 139.7)
-		)
-		(stroke
-			(width 0)
-			(type default)
-		)
-	)
-	(wire
-		(pts
 			(xy 24.13 49.53) (xy 30.48 49.53)
 		)
@@
 		)
 	)
-	(wire
-		(pts
-			(xy 102.87 134.62) (xy 102.87 139.7)
-		)
-		(stroke
-			(width 0)
-			(type default)
-		)
-	)
 	(bus
 		(pts
@@
 		)
 	)
-	(label "BIAS_SHD"
-		(at 41.91 88.9 180)
-		(effects
-			(font
-				(size 1.27 1.27)
-			)
-			(justify right bottom)
-		)
-	)
 	(label "IN_ELEC"
 		(at 35.56 35.56 0)
@@
 		)
 	)
-	(hierarchical_label "BIAS_SHD"
-		(shape input)
-		(at 31.75 88.9 180)
-		(effects
-			(font
-				(size 1.27 1.27)
-			)
-			(justify right)
-		)
-	)
 	(hierarchical_label "IN8+"
 		(shape output)
@@
 	)
 	(symbol
-		(lib_name "TPD4E001DPKT_1")
 		(lib_id "TPD4:TPD4E001DPKT")
 		(at 102.87 107.95 270)
@@
 		)
 		(property "Footprint" "DPK6"
-			(at 105.41 107.95 0)
+			(at 112.268 120.65 0)
 			(hide yes)
 			(show_name no)
@@
 			)
 		)
-		(property "Datasheet" "${DSH}/protection/tpd4e001.pdf"
-			(at 105.41 106.68 0)
+		(property "Datasheet" "https://www.ti.com/lit/gpn/tpd4e001"
+			(at 109.982 119.888 0)
 			(hide yes)
 			(show_name no)
@@
 	)
 	(symbol
-		(lib_name "TPD4E001DPKT_1")
 		(lib_id "TPD4:TPD4E001DPKT")
 		(at 102.87 46.99 270)
@@
 			)
 		)
-		(property "Datasheet" "${DSH}/protection/tpd4e001.pdf"
+		(property "Datasheet" "https://www.ti.com/lit/gpn/tpd4e001"
 			(at 105.41 45.72 0)
 			(hide yes)
@@
 	)
 	(symbol
-		(lib_name "TPD4E001DPKT_1")
 		(lib_id "TPD4:TPD4E001DPKT")
 		(at 205.74 81.28 270)
@@
 			)
 		)
-		(property "Datasheet" "${DSH}/protection/tpd4e001.pdf"
+		(property "Datasheet" "https://www.ti.com/lit/gpn/tpd4e001"
 			(at 208.28 80.01 0)
 			(hide yes)

Commit message: replanteo de conectores
Parts:
- added C14, C16, C17, C18: 1nF, Capacitor_SMD:C_0603_1608Metric, symbol Device:C
- added R12, R13, R15, R20: 2k2, Resistor_SMD:R_0603_1608Metric, symbol Device:R
- added U10, U11, U5: TPD4E001, Power:DPK6, symbol TPD4:TPD4E001DPKT
- C1, C10, C11, C12, C34, C5, C6, C7, C8, C9: footprint (none) -> Capacitor_SMD:C_0603_1608Metric
- R10, R11, R18, R19, R21, R4, R5, R6, R7, R8, R9: footprint (none) -> Resistor_SMD:R_0603_1608Metric
- U3, U4, U8: footprint DPK6 -> Power:DPK6
Connections:
- net AGND: now also C14.2, C16.2, C17.2, C18.2
- net AVDD: now also U11.6 (VCC)
- net AVSS: now also U11.3 (GND)
- net CH_IN5: now also R20.2, U11.1 (IO1)
- net CH_IN6: now also R13.2, U11.2 (IO2)
- net CH_IN7: now also R12.2, U11.4 (IO3)
- net CH_IN8: now also R15.2, U11.5 (IO4)
- net IN5+: now also C17.1, R20.1
- net IN6+: now also C14.1, R13.1
- net IN7+: now also C16.1, R12.1
- net IN8+: now also C18.1, R15.1
Other:
- moved on the sheet: C1, C34, R18, R19, R21, U8
