File: PCB/submodule/ads1299.kicad_sch (KiCad schematic)
At the start: 63 parts, among them J1 Conn_01x01_Pin, J10 Conn_01x01_Pin, J11 Conn_01x01_Pin, J18 Conn_01x01_Pin, J19 Conn_01x01_Pin, J2 Conn_01x01_Pin, J3 Conn_01x01_Pin, J4 Conn_01x01_Pin, J5 Conn_01x01_Pin, J8 Conn_01x01_Pin, U1 ADS1299IPAG, U2 OPA2376, U5 OPA2376xxD

Commit message: ECR ok
Parts:
- removed C14, C16, C17, C18, C19, C20, C21, C22: 4.7uF, symbol Device:C
- removed J1, J18, J19, J2, J3, J4, J5, J8: Conn_01x01_Pin, symbol Connector:Conn_01x01_Pin
- removed JP10, JP11, JP12, JP13, JP14, JP15, JP8, JP9: SolderJumper_2_Bridged, symbol Jumper:SolderJumper_2_Bridged
- removed JP17: SB_BIASREF, symbol Jumper:SolderJumper_2_Open
- removed U2: OPA2376, symbol Device:Opamp_Dual
- removed U5: OPA2376xxD, symbol Amplifier_Operational:OPA2376xxD
- added C45, C46, C47, C48, C49, C50, C51, C52: 4.7uF, symbol Device:C
- added J12, J16, J17, J20, J21, J22, J23, J7: Conn_01x01_Pin, symbol Connector:Conn_01x01_Pin
- added JP16, JP17, JP18, JP19, JP20, JP21, JP22, JP23: SolderJumper_2_Bridged, symbol Jumper:SolderJumper_2_Bridged
- added U9: OPA2376xxD, Package_SO:SO-20-1EP_7.52x12.825mm_P1.27mm_EP6.045x12.09mm_Mask3.56x4.47mm, symbol Amplifier_Operational:OPA2376xxD
Connections:
- net DVDD is gone; now on net +3.3V: C35.1, C36.1, R14.2, R16.2, U1.48 (DVDD), U1.50 (DVDD)
- net AGND: now also C43.2, C44.2, JP16.1 (A), JP17.1 (A), JP18.1 (A), JP19.1 (A), JP20.1 (A), JP21.1 (A), JP22.1 (A), JP23.1 (A)
- net AVDD: now also C15.1, U1.54 (AVDD1), U9.8 (V+)
- net AVSS: now also U9.4 (V-)
- net BIASINV_LINK: no longer U1.37 (CLK)
- net BIAS_SHD: now also U9.6 (-), U9.7
- net IN1-: now also C47.2, J21.1 (Pin_1), JP18.2 (B)
- net IN2-: now also C45.2, J20.1 (Pin_1), JP16.2 (B)
- net IN3-: now also C48.2, J12.1 (Pin_1), JP19.2 (B)
- net IN4-: now also C46.2, J7.1 (Pin_1), JP17.2 (B)
- net IN5-: now also C51.2, J23.1 (Pin_1), JP22.2 (B)
- net IN6-: now also C49.2, J22.1 (Pin_1), JP20.2 (B)
- net IN7-: now also C52.2, J17.1 (Pin_1), JP23.2 (B)
- net IN8-: now also C50.2, J16.1 (Pin_1), JP21.2 (B)
- net IN_REF: now also U9.3 (+)
- net at U1.60 (BIASREF): now also J11.1 (Pin_1)
- net at JP6.1 (A): now also U9.1, U9.2 (-)
- net at R2.2: now also U9.5 (+)
- new net: C51.1, C52.1
- new net: C45.1, C46.1
- new net: C47.1, C48.1
- new net: C49.1, C50.1
- new net CLK: U1.37 (CLK)
Other:
- note removed: "SB_BIASREF: - BASE = Open (default) - EXP = Open (default)"
- moved on the sheet: J11, JP4

Commit message: replanteo de conectores
Parts:
- removed C45, C46, C47, C48, C49, C50, C51, C52: 4.7uF, symbol Device:C
- removed J12, J16, J17, J20, J21, J22, J23, J7: Conn_01x01_Pin, symbol Connector:Conn_01x01_Pin
- removed JP16, JP17, JP18, JP19, JP20, JP21, JP22, JP23: SolderJumper_2_Bridged, symbol Jumper:SolderJumper_2_Bridged
- C13, C15, C2, C29, C3, C31, C32, C35, C36, C37, C38, C39, C4, C40, C41, C42, C43, C44: footprint (none) -> Capacitor_SMD:C_0603_1608Metric
- C30: footprint (none) -> Capacitor_SMD:C_0805_2012Metric
- C33: footprint (none) -> Capacitor_SMD:C_1210_3225Metric
- J10, J11: footprint (none) -> Connector_PinHeader_2.54mm:PinHeader_1x01_P2.54mm_Vertical
- JP1, JP2, JP3: footprint (none) -> Jumper:SolderJumper-3_P2.0mm_Open_TrianglePad1.0x1.5mm_NumberLabels
- JP4, JP5, JP7: footprint (none) -> Jumper:SolderJumper-2_P1.3mm_Open_TrianglePad1.0x1.5mm
- JP6: footprint (none) -> Jumper:SolderJumper-3_P1.3mm_Bridged12_Pad1.0x1.5mm_NumberLabels
- R1, R14, R16, R17, R2, R3: footprint (none) -> Resistor_SMD:R_0603_1608Metric
- U1: footprint PAG64_TEX -> Power:PAG64_TEX
Other:
- note added: "Agregar protecciones para canales - - GPIOs analogicos o digitales?"
- note added: "El electrodo del bias debe pasar por el seguidor?"
- note removed: "Optional Differential Inputs"
- moved on the sheet: J10, J11, R14
