File: PCB/submodule/submodule.kicad_sch (KiCad schematic)
At the start: 25 parts, among them J13 CONN_SUBMODULES, J24 MAIN, J32 Conn_Coaxial, J33 Conn_Coaxial, J34 ELECT_AUX, J35 Conn_Coaxial, J36 Conn_Coaxial, J37 Conn_Coaxial, J38 Conn_Coaxial, J39 Conn_Coaxial, J40 Conn_Coaxial, J41 Conn_Coaxial, J42 Conn_Coaxial, J6 GPIOs, J9 Conn_01x06, U6 LP5907, U7 TPS72325

Commit message: ECR ok
Parts:
- removed JP16: SB_GND_TIE, symbol Jumper:SolderJumper_2_Open
- removed TP1: TestPoint, symbol Connector:TestPoint
- added L3, L4, L5: HZ0805E601R-10, Package_TO_SOT_SMD:SOT-23-5, symbol Device:L
Connections:
- net +3.3V: now also L4.1; no longer C23.1, J9.7 (Pin_7), U6.1 (VIN), U6.3 (EN)
- net -3V3: now also L5.1; no longer C27.1, U7.2 (IN), U7.3 (EN)
- net AGND: now also L3.2; no longer J24.12 (Pin_12)
- net DGND: now also J24.12 (Pin_12), J9.7 (Pin_7), L3.1
- new net: C23.1, L4.2, U6.1 (VIN), U6.3 (EN)
- new net: C27.1, L5.2, U7.2 (IN), U7.3 (EN)
Other:
- sheet PROTECCIONES ports: added none; removed BIAS_SHD
- note added: "agregar test points"
- note added: "cambiar por 2x6"
- note added: "separar DIGITAL & ANALOG ARRIBA Y ABAJO"
- moved on the sheet: C23, C24, C25, C26, C27, C28, J9, U6, U7

Commit message: replanteo de conectores
Parts:
- removed J24: MAIN, symbol Connector_Generic:Conn_02x07_Odd_Even
- removed J9: Conn_01x06, symbol Connector_Generic:Conn_01x08
- added J1: MAIN, Connector:Tag-Connect_TC2030-IDC-FP_2x03_P1.27mm_Vertical, symbol Connector_Generic:Conn_02x04_Odd_Even
- added J43: ELECT-_AUX, Connector_PinHeader_2.54mm:PinHeader_1x12_P2.54mm_Vertical, symbol Connector_Generic:Conn_01x12
- C23, C24, C25, C27, C28: footprint (none) -> Capacitor_SMD:C_0603_1608Metric
- C26: footprint (none) -> Capacitor_SMD:C_0805_2012Metric
- J13: footprint (none) -> Connector_PinHeader_2.54mm:PinHeader_1x09_P2.54mm_Vertical
- J34: value ELECT_AUX -> ELECT+_AUX; footprint (none) -> Connector_PinHeader_2.54mm:PinHeader_1x12_P2.54mm_Vertical
- J6: footprint (none) -> Connector_PinHeader_2.54mm:PinHeader_1x04_P2.54mm_Vertical; symbol Connector_Generic:Conn_01x04 -> Connector_Generic:Conn_01x06
Connections:
- net PWDN is gone; now on net DGND: J13.18 (Pin_18)
- net +3.3V: now also J6.1 (Pin_1), J1.1 (Pin_1)
- net -3V3: now also J1.2 (Pin_2)
- net ADS1299/GPIO1: now also J6.2 (Pin_2); no longer J6.1 (Pin_1)
- net ADS1299/GPIO2: now also J6.3 (Pin_3); no longer J6.2 (Pin_2)
- net ADS1299/GPIO3: now also J6.4 (Pin_4); no longer J6.3 (Pin_3)
- net ADS1299/GPIO4: now also J6.5 (Pin_5); no longer J6.4 (Pin_4)
- net AGND: now also J43.10 (Pin_10), J43.11 (Pin_11), J43.12 (Pin_12), J43.9 (Pin_9)
- net CLK: now also J13.14 (Pin_14); no longer J13.15 (Pin_15)
- net CS: now also J1.6 (Pin_6)
- net DGND: now also J6.6 (Pin_6), J1.8 (Pin_8); no longer J13.10 (Pin_10), J13.13 (Pin_13), J13.17 (Pin_17)
- net DRDY_OUT: now also J1.4 (Pin_4)
- net MISO: now also J1.7 (Pin_7)
- net MOSI: now also J1.5 (Pin_5)
- net RESET: no longer J13.16 (Pin_16)
- net SCLK: now also J1.3 (Pin_3)
- net START: no longer J13.14 (Pin_14)
- net CH_IN1 renamed CH_IN1+
- net CH_IN2 renamed CH_IN2+
- net CH_IN3 renamed CH_IN3+
- net CH_IN4 renamed CH_IN4+
- net CH_IN5 renamed CH_IN5+
- net CH_IN6 renamed CH_IN6+
- net CH_IN7 renamed CH_IN7+
- net CH_IN8 renamed CH_IN8+
- new net CH_IN1-: J43.1 (Pin_1)
- new net CH_IN2-: J43.2 (Pin_2)
- new net CH_IN3-: J43.3 (Pin_3)
- new net CH_IN4-: J43.4 (Pin_4)
- new net CH_IN5-: J43.5 (Pin_5)
- new net CH_IN6-: J43.6 (Pin_6)
- new net CH_IN7-: J43.7 (Pin_7)
- new net CH_IN8-: J43.8 (Pin_8)
Other:
- sheet ADS1299 ports: added IN1-, IN2-, IN3-, IN4-, IN5-, IN6-, IN7-, IN8-; removed PWDN
- sheet PROTECCIONES ports: added CH_IN+[1..8], IN1-, IN2-, IN3-, IN4-, IN5-, IN6-, IN7-, IN8-; removed CH_IN[1..8]
- note added: "Depende del espacio"
- note removed: "Debug Access"
- note removed: "cambiar por 2x6"
- moved on the sheet: J34, J35, J36, J37, J38, J39, J40, J41, J42, L3
